File: placa_iot/alimentacion.kicad_sch (KiCad schematic)
At the start: 0 parts

Commit message: Alimetación creada
Parts:
- added C2, C3, C4, C5: 100 nF, Capacitor_SMD:C_0402_1005Metric, symbol Device:C
- added R1, R2, R3: 10 kOhm, Resistor_SMD:R_0402_1005Metric, symbol Device:R
- added U1, U2: RT9080-33GJ5, ic_power:TSOT-23-5_RIT, symbol ic_power:RT9080-33GJ5
Connections:
- new net: R2.2, R3.2, U2.3 (EN)
- new net: R1.2, U1.3 (EN)
- new net +3.3V: C5.1, U1.5 (VOUT)
- new net +5V: C2.1, C3.1, R1.1, R2.1, U1.1 (VIN), U2.1 (VIN)
- new net GND: C2.2, C3.2, C4.2, C5.2, U1.2 (GND), U2.2 (GND)
- new net Vcc+3.3: C4.1, U2.5 (VOUT)

Commit message: Microcontrolador en proceso
Parts:
- R3: value 10 kOhm -> 0 Ohm
Connections:
- net IO35: now reaches R3.1
Changed lines of the file:
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@@
+	(wire
+		(pts
+			(xy 142.24 78.74) (xy 142.24 83.82)
+		)
+		(stroke
+			(width 0)
+			(type default)
+		)
+	)
 	(wire
 		(pts
@@
 			(width 0)
 			(type default)
+		)
+	)
+	(global_label "IO35"
+		(shape input)
+		(at 142.24 83.82 270)
+		(fields_autoplaced yes)
+		(effects
+			(font
+				(size 1.27 1.27)
+			)
+			(justify right)
+		)
+		(property "Intersheetrefs" "${INTERSHEET_REFS}"
+			(at 142.24 91.1595 90)
+			(hide yes)
+			(show_name no)
+			(do_not_autoplace no)
+			(effects
+				(font
+					(size 1.27 1.27)
+				)
+				(justify right)
+			)
 		)
 	)
@@
 			)
 		)
-		(property "Value" "10 kOhm"
-			(at 139.7 72.39 90)
-			(show_name no)
-			(do_not_autoplace no)
+		(property "Value" "0 Ohm"
+			(at 139.7 74.422 90)
+			(show_name no)
+			(do_not_autoplace no)

Commit message: Esquemático acabado
Changed lines of the file:
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@@
 		)
 	)
-	(global_label "IO35"
+	(hierarchical_label "IO35"
 		(shape input)
 		(at 142.24 83.82 270)
-		(fields_autoplaced yes)
 		(effects
 			(font
@@
 			(justify right)
 		)
-		(property "Intersheetrefs" "${INTERSHEET_REFS}"
-			(at 142.24 91.1595 90)
-			(hide yes)
-			(show_name no)
-			(do_not_autoplace no)
-			(effects
-				(font
-					(size 1.27 1.27)
-				)
-				(justify right)
-			)
-		)
 	)
