File: placa_iot/battery.kicad_sch (KiCad schematic)
At the start: 0 parts

Commit message: Batería completa
Parts:
- added C26, C28: 100 nF, Capacitor_SMD:C_0402_1005Metric, symbol Device:C
- added C27, C29: 10 uF, Capacitor_SMD:C_0402_1005Metric, symbol Device:C
- added D1, D4: SS34, Diode_SMD:D_SMA, symbol Diode:SS34
- added D2: BLUE, LED_SMD:LED_0402_1005Metric, symbol Device:LED
- added D3: DZ 5.6V, Diode_SMD:D_SOD-123, symbol Device:D_Zener
- added D5: RED, LED_SMD:LED_0402_1005Metric, symbol Device:LED
- added J4: 620102131822, connectors:CONN_SMT_MH_SH_P2.00MM_P2, symbol connectors:CONN_SMT_MH_SH_P2.00MM_P2
- added J6: B2B-PH-K-S(LF)(SN), connectors:CONN_THT_MV_JST_P2.00MM_P2, symbol connectors:CONN_THT_MV_JST_P2.00MM_P2
- added Q1, Q2: Q_PMOS, Package_TO_SOT_SMD:SOT-23, symbol Device:Q_PMOS
- added R14, R15, R16, R17: 100K 1%, Resistor_SMD:R_0402_1005Metric, symbol Device:R
- added R18, R19: 1k, Resistor_SMD:R_0402_1005Metric, symbol Device:R
- added R20: 2k, Resistor_SMD:R_0402_1005Metric, symbol Device:R
- added R21: 0, Resistor_SMD:R_0402_1005Metric, symbol Device:R
- added R9: 10k, Resistor_SMD:R_0402_1005Metric, symbol Device:R
- added SW3: SW_SPDT, symbol Switch:SW_SPDT
- added U6: CN3065, ic_power:DFN-8-1EP_3x3mm_P0.5mm_EP1.66x2.38mm, symbol ic_power:CN3065
Connections:
- new net: C27.1, C28.1, D4.1 (K), Q2.S, R18.2, R19.2, U6.4 (VIN)
- new net: R21.2, U6.1 (TEMP)
- new net: R20.2, U6.2 (ISET)
- new net: D2.1 (K), U6.6 (~{DONE})
- new net: D5.1 (K), U6.7 (~{CHRG})
- new net: D2.2 (A), R18.1
- new net: D1.1 (K), Q1.S, SW3.2 (B)
- new net: D5.2 (A), R19.1
- new net +5V: SW3.1 (A)
- new net GND: C26.2, C27.2, C28.2, C29.2, D3.2 (A), J4.2 (Pin_2), J6.2 (Pin_2), R15.1, R17.1, R20.1, R21.1, R9.1, U6.3 (GND), U6.9 (GND)
- new net IO1: C26.1, R14.1, R15.2
- new net IO4: R16.1, R17.2
- new net VBAT: C29.1, J4.1 (Pin_1), Q1.D, R14.2, U6.5 (BAT), U6.8 (FB)
- new net VBUS: D1.2 (A), D4.2 (A), Q1.G, Q2.G, R9.2
- new net VSOLAR: D3.1 (K), J6.1 (Pin_1), Q2.D, R16.2
- no-connect marks 0 -> 3

Commit message: Esquemático acabado
Changed lines of the file:
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@@
 	)
 	(hierarchical_label "IO4"
-		(shape bidirectional)
+		(shape output)
 		(at 167.64 149.86 180)
 		(effects

Commit message: Layout iniciado y resolución de errores de huellas
Parts:
- removed Q2: Q_PMOS, Package_TO_SOT_SMD:SOT-23, symbol Device:Q_PMOS
- added Q3: Q_PMOS, Package_TO_SOT_SMD:SOT-23, symbol Device:Q_PMOS
- J4: footprint connectors:CONN_SMT_MH_SH_P2.00MM_P2 -> Connectors:CONN_SMT_MH_SH_P2.00MM_P2
- J6: footprint connectors:CONN_THT_MV_JST_P2.00MM_P2 -> Connectors:CONN_THT_MV_JST_P2.00MM_P2
- SW3: footprint (none) -> Button_Switch_THT:SW_Slide_SPDT_Angled_CK_OS102011MA1Q
Connections:
- net VBAT: now also Q1.3 (D); no longer Q1.D
- net VBUS: now also Q1.1 (G), Q3.1 (G); no longer Q1.G
- net VSOLAR: now also Q3.3 (D)
- net at C27.1, C28.1, D4.1 (K)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: now also Q3.2 (S)
- net at D1.1 (K), SW3.2 (B): now also Q1.2 (S); no longer Q1.S
Changed lines of the file:
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@@
 			)
 		)
-		(property "Footprint" "connectors:CONN_SMT_MH_SH_P2.00MM_P2"
+		(property "Footprint" "Connectors:CONN_SMT_MH_SH_P2.00MM_P2"
 			(at 426.72 101.6 0)
 			(hide yes)
@@
 	)
 	(symbol
+		(lib_name "Q_PMOS_1")
 		(lib_id "Device:Q_PMOS")
 		(at 76.2 133.35 0)
@@
 			)
 		)
-		(pin "S"
-		)
-		(pin "D"
-		)
-		(pin "G"
+		(pin "1"
+		)
+		(pin "3"
+		)
+		(pin "2"
 		)
 		(instances
@@
 				(path "/ca8a6ff9-ef79-4432-921e-b6a14ecba63b/8dc7ab2b-7411-4406-b884-e10648d74030"
 					(reference "Q1")
+					(unit 1)
+				)
+			)
+		)
+	)
+	(symbol
+		(lib_name "Q_PMOS_1")
+		(lib_id "Device:Q_PMOS")
+		(at 203.2 133.35 90)
+		(unit 1)
+		(body_style 1)
+		(exclude_from_sim no)
+		(in_bom yes)
+		(on_board yes)
+		(in_pos_files yes)
+		(dnp no)
+		(fields_autoplaced yes)
+		(property "Reference" "Q3"
+			(at 203.2 124.46 90)
+			(show_name no)
+			(do_not_autoplace no)
+			(effects
+				(font
+					(size 1.27 1.27)
+				)
+			)
+		)
+		(property "Value" "Q_PMOS"
+			(at 203.2 127 90)
+			(show_name no)
+			(do_not_autoplace no)
+			(effects
+				(font
+					(size 1.27 1.27)
+				)
+			)
+		)
+		(property "Footprint" "Package_TO_SOT_SMD:SOT-23"
+			(at 200.66 128.27 0)
+			(hide yes)
+			(show_name no)
+			(do_not_autoplace no)
+			(effects
+				(font
+					(size 1.27 1.27)
+				)
+			)
+		)
+		(property "Datasheet" ""
+			(at 203.2 133.35 0)
+			(hide yes)
+			(show_name no)
+			(do_not_autoplace no)
+			(effects
+				(font
+					(size 1.27 1.27)
+				)
+			)
+		)
+		(property "Description" "P-MOSFET transistor"
+			(at 203.2 133.35 0)
+			(hide yes)
+			(show_name no)
+			(do_not_autoplace no)
+			(effects
+				(font
+					(size 1.27 1.27)
+				)
+			)
+		)
+		(pin "1"
+		)
+		(pin "3"
+		)
+		(pin "2"
+		)
+		(instances
+			(project "placa_iot"
+				(path "/ca8a6ff9-ef79-4432-921e-b6a14ecba63b/8dc7ab2b-7411-4406-b884-e10648d74030"
+					(reference "Q3")
 					(unit 1)
 				)
@@
 			)
 		)
-		(property "Footprint" ""
+		(property "Footprint" "Button_Switch_THT:SW_Slide_SPDT_Angled_CK_OS102011MA1Q"
 			(at 78.74 157.48 0)
 			(hide yes)
@@
 	)
 	(symbol
-		(lib_id "Device:Q_PMOS")
-		(at 203.2 133.35 90)
-		(unit 1)
-		(body_style 1)
-		(exclude_from_sim no)
-		(in_bom yes)
-		(on_board yes)
-		(in_pos_files yes)
-		(dnp no)
-		(fields_autoplaced yes)
-		(property "Reference" "Q2"
-			(at 203.2 124.46 90)
-			(show_name no)
-			(do_not_autoplace no)
-			(effects
-				(font
-					(size 1.27 1.27)
-				)
-			)
-		)
-		(property "Value" "Q_PMOS"
-			(at 203.2 127 90)
-			(show_name no)
-			(do_not_autoplace no)
-			(effects
-				(font
-					(size 1.27 1.27)
-				)
-			)
-		)
-		(property "Footprint" "Package_TO_SOT_SMD:SOT-23"
-			(at 200.66 128.27 0)
-			(hide yes)
-			(show_name no)
-			(do_not_autoplace no)
-			(effects
-				(font
-					(size 1.27 1.27)
-				)
-			)
-		)
-		(property "Datasheet" ""
-			(at 203.2 133.35 0)
-			(hide yes)
-			(show_name no)
-			(do_not_autoplace no)
-			(effects
-				(font
-					(size 1.27 1.27)
-				)
-			)
-		)
-		(property "Description" "P-MOSFET transistor"
-			(at 203.2 133.35 0)
-			(hide yes)
-			(show_name no)
-			(do_not_autoplace no)
-			(effects
-				(font
-					(size 1.27 1.27)
-				)
-			)
-		)
-		(pin "S"
-		)
-		(pin "D"
-		)
-		(pin "G"
-		)
-		(instances
-			(project "placa_iot"
-				(path "/ca8a6ff9-ef79-4432-921e-b6a14ecba63b/8dc7ab2b-7411-4406-b884-e10648d74030"
-					(reference "Q2")
-					(unit 1)
-				)
-			)
-		)
-	)
-	(symbol
 		(lib_id "Device:LED")
 		(at 260.35 149.86 90)
@@
 			)
 		)
-		(property "Footprint" "connectors:CONN_THT_MV_JST_P2.00MM_P2"
+		(property "Footprint" "Connectors:CONN_THT_MV_JST_P2.00MM_P2"
 			(at 114.3 100.33 0)
 			(hide yes)
