File: placa_iot/rf.kicad_sch (KiCad schematic)
At the start: 0 parts

Commit message: RF completado
Parts:
- added C23, C24, C25: NC, Capacitor_SMD:C_0402_1005Metric, symbol Device:C
- added J3: 20279-001E-03, antennas:IPEX_MHF_I, symbol Antenas:IPEX_MHF_I
- added R10, R11, R12, R13: 22 Ohm, Resistor_SMD:R_0402_1005Metric, symbol Device:R
- added U5: T-SX1262, ic_control:MODULE_T_SX1262, symbol ic_control:T_SX1262
Connections:
- new net: R11.2, U5.10 (DIO1)
- new net: R12.2, U5.13 (NC)
- new net: R13.2, U5.14 (DIO3)
- new net: C23.1, C24.1, U5.16 (ANT)
- new net: R10.2, U5.9 (BUSY)
- new net: C24.2, C25.1, J3.1 (In)
- new net GND: C23.2, C25.2, J3.2 (Ext), J3.3 (Ext), U5.1 (GND), U5.15 (GND), U5.8 (GND)
- new net IO3: U5.7 (MISO)
- new net IO33: R11.1
- new net IO34: R10.1
- new net IO36: U5.2 (NC)
- new net IO5: U5.5 (SCK)
- new net IO6: U5.6 (MOSI)
- new net IO7: U5.4 (NSS)
- new net IO8: U5.3 (NRESET)
- new net IO9: U5.11 (NC)
- new net LORA_RX: R13.1
- new net LORA_TX: R12.1
- new net Vcc+3.3: U5.12 (3.3V)

Commit message: Layout iniciado y resolución de errores de huellas
Parts:
- J3: footprint antennas:IPEX_MHF_I -> Antennas:IPEX_MHF_I
Changed lines of the file:
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@@
 			)
 		)
-		(property "Footprint" "antennas:IPEX_MHF_I"
+		(property "Footprint" "Antennas:IPEX_MHF_I"
 			(at 314.96 46.99 0)
 			(hide yes)
