File: placa_iot/microcontrolador.kicad_sch (KiCad schematic)
At the start: 33 parts, among them J1 22-28-4144, J2 22-28-4144, SW1 RST/EN, SW2 BOOT, U3 ESP32-S3, U4 PRO-OB-536, Y1 40 MHz

Commit message: Colocación de elementos
Connections:
- net LNA: now reaches C16.1, C17.1, C18.1, C18.2, C19.1, C20.1, U3.1 (LNA_IN)
Changed lines of the file:
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@@
+		)
+	)
+	(label "LNA"
+		(at 243.84 176.53 180)
+		(effects
+			(font
+				(size 1.27 1.27)
+			)
+			(justify right bottom)
 		)
 	)
