File: placa_iot/placa_iot.kicad_pcb (KiCad board)
At the start: 4 copper layers, 84 parts, among them J1 22-28-4144, J2 22-28-4144, J3 20279-001E-03, J4 620102131822, J5 USB4105-GF-A-120, J6 B2B-PH-K-S(LF)(SN), Q1 Q_PMOS, Q3 Q_PMOS, SW1 RST/EN, SW2 BOOT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

Commit message: Colocación de elementos
Parts:
- added M1: MountingHole_2.5mm_Pad, MountingHole:MountingHole_2.5mm_Pad, F.Cu at (30.0, 55.0)
- added M2: MountingHole_2.5mm_Pad, MountingHole:MountingHole_2.5mm_Pad, F.Cu at (68.9, 55.0)
- added M3: MountingHole_2.5mm_Pad, MountingHole:MountingHole_2.5mm_Pad, F.Cu at (30.0, 165.0)
- added M4: MountingHole_2.5mm_Pad, MountingHole:MountingHole_2.5mm_Pad, F.Cu at (68.9, 165.0)
- J1, J2: moved to B.Cu
- moved C25 127.9 mm to (35.0, 135.9), turned to 90 degrees
- moved C24 126.7 mm to (36.5, 135.9), turned to -90 degrees
- moved C23 125.5 mm to (38.1, 135.9), turned to -90 degrees
- moved C26 123.7 mm to (52.3, 147.3), turned to 180 degrees
- moved C29 118.5 mm to (52.3, 143.4), turned to 180 degrees
- moved D3 118.4 mm to (64.0, 156.1), turned to -90 degrees
- moved U5 118.3 mm to (41.9, 102.9), turned to 180 degrees
- moved C27 116.5 mm to (61.6, 149.8)
- moved C28 116.0 mm to (61.6, 151.0)
- moved J6 115.8 mm to (69.6, 152.5), turned to -90 degrees
- moved J3 115.3 mm to (29.0, 136.5), turned to 90 degrees
- moved J4 114.2 mm to (56.5, 164.5)
- moved R20 113.8 mm to (56.1, 149.7), turned to 180 degrees
- moved R10 113.5 mm to (48.3, 100.1), turned to -90 degrees
- moved R21 113.5 mm to (56.1, 151.0), turned to 180 degrees
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Connections:
- net Net-(U3-LNA_IN) renamed /MICROCONTROLADOR/LNA
Other:
- board outline added: 48.6 x 120 mm

Commit message: Layout Completado
Parts:
- moved C3 65.7 mm to (38.0, 122.3), turned to 180 degrees
- moved R3 62.5 mm to (38.0, 125.0), turned to 0 degrees
- moved U2 61.3 mm to (41.8, 124.0), turned to 0 degrees
- moved C4 60.4 mm to (45.6, 122.9), turned to 0 degrees
- moved R2 60.2 mm to (38.0, 123.6), turned to 180 degrees
- moved C2 47.0 mm to (55.5, 122.7), turned to 0 degrees
- moved C5 45.0 mm to (63.3, 121.9), turned to 0 degrees
- moved R1 41.8 mm to (55.5, 124.0), turned to 0 degrees
- moved U1 38.4 mm to (59.4, 122.9), turned to 0 degrees
- moved D7 8.89 mm to (44.5, 157.8), turned to -90 degrees
- moved R24 6.79 mm to (37.2, 157.7)
- moved R26 5.92 mm to (43.1, 157.7), turned to -90 degrees
- moved FL1 2.93 mm to (41.6, 157.4), turned to 180 degrees
- moved R25 2.41 mm to (40.1, 157.7), turned to -90 degrees
- moved D8 2.14 mm to (38.7, 157.8)
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